Commit message: yaw control

File: src/cmg_leg_description/urdf/cmg_joint.urdf (robot description, URDF)
Before this commit: robot wheeled_inverted_pendulum, 11 links, 10 joints
Joints:
- joint ankle_pitch_joint: origin xyz=0 0 0.0 rpy=0.0 0.490655767230835 0.0 -> xyz=0 0 0.0 rpy=0.0 0.745238866846359 0.0
- joint hip_pitch_joint: origin xyz=0 0 0.28 rpy=0.0 0.568004838041421 0.0 -> xyz=0 0 0.28 rpy=0.0 0.885462876712376 0.0
- joint imu_joint: axis 0 0 1 -> (none); limit lower=0.0 upper=0 effort=1000 velocity=1000 -> (none); type revolute -> fixed
- joint knee_joint: origin xyz=0 0 0.279942 rpy=0.0 -1.05866060527226 0.0 -> xyz=0 0 0.279942 rpy=0.0 -1.63070174355873 0.0
